Commit message: use official urdf & add tool link

File: elfin3/elfin3_ros2_gazebo/urdf/elfin3.urdf.xacro (robot description, xacro)
@@ -4,16 +4,16 @@
   <xacro:arg name="use_fake_hardware" default="false" />
   <!-- Load TRANSMISSION file: -->
-  <xacro:include filename="$(find elfin3_ros2_gazebo)/urdf/elfin3_transmission.xacro" />
+  <!-- <xacro:include filename="$(find elfin3_ros2_gazebo)/urdf/elfin3_transmission.xacro" /> -->
   <!-- Load GAZEBO/ROS2_CONTROL file: -->
-  <xacro:include filename="$(find elfin3_ros2_gazebo)/urdf/elfin3_gazebo.xacro" />
+  <!-- <xacro:include filename="$(find elfin3_ros2_gazebo)/urdf/elfin3_gazebo.xacro" /> -->
   <xacro:property name="PI" value="3.1415926535897931"/>
   <xacro:property name="density" value="3.09"/>
   <!-- <xacro:macro name="elfin3"> -->
     <!-- TRANSMISSION: -->
-    <xacro:elfin3_transmission />
+    <!-- <xacro:elfin3_transmission /> -->
     <!-- GAZEBO - ROS2_CONTROL: -->
-    <xacro:elfin3_gazebo
+    <!-- <xacro:elfin3_gazebo
     use_real_hardware="$(arg use_real_hardware)"
-    use_fake_hardware="$(arg use_fake_hardware)"/>
+    use_fake_hardware="$(arg use_fake_hardware)"/> -->
   <link name="world"/>
   <joint name="world_base" type="fixed">
@@ -439,13 +439,27 @@
       xyz="0 0 0" />
   </joint>
-  <link name="elfin_dummy_gripper"/>
-  <joint name="elfin_dummy_joint" type="fixed">
-    <origin
-      xyz="0 -0.111 0"
-      rpy="${PI/2} ${-PI/2} 0" />
-    <parent
-      link="elfin_link6" />
-    <child
-      link="elfin_dummy_gripper" />
-  </joint>
+  <!-- Add tool link -->
+<link name="tool_link">
+  <visual>
+    <origin xyz="0 0 0" rpy="0 0 0"/>
+    <!-- <geometry>
+      <mesh filename="file://$(find your_package)/meshes/tool.stl"/>
+    </geometry> -->
+    <material name="tool_color">
+      <color rgba="0.8 0.2 0.2 1.0"/>
+    </material>
+  </visual>
+  <collision>
+    <origin xyz="0 0 0" rpy="0 0 0"/>
+    <!-- <geometry>
+      <mesh filename="file://$(find your_package)/meshes/tool.stl"/>
+    </geometry> -->
+  </collision>
+</link>
+<!-- Add tool joint -->
+<joint name="tool_joint" type="fixed">
+  <origin xyz="0 0 0.11" rpy="0 0 0"/>  <!-- 沿Z轴偏移110mm -->
+  <parent link="elfin_end_link"/>
+  <child link="tool_link"/>
+</joint>
 </robot>

File: elfin_description/urdf/elfin3.urdf.xacro (robot description, xacro)
@@ -1,19 +1,9 @@
-<?xml version="1.0"?>
-<robot name="elfin3" xmlns:xacro="http://wiki.ros.org/xacro">
-  <xacro:arg name="use_real_hardware" default="false" />
-  <xacro:arg name="use_fake_hardware" default="true" />
-  <!-- Load TRANSMISSION file: -->
-  <!-- <xacro:include filename="$(find elfin3_ros2_gazebo)/urdf/elfin3_transmission.xacro" /> -->
-  <!-- Load GAZEBO/ROS2_CONTROL file: -->
-  <!-- <xacro:include filename="$(find elfin3_ros2_gazebo)/urdf/elfin3_gazebo.xacro" /> -->
+<robot
+  name="elfin3" xmlns:xacro="http://www.ros.org/wiki/xacro">
+  <xacro:include filename="$(find elfin_description)/urdf/materials.xacro" />
+  <!-- <xacro:include filename="$(find elfin_description)/urdf/elfin_robot.gazebo" /> -->
+  <xacro:include filename="$(find elfin_description)/urdf/elfin_transmission.xacro" />
   <xacro:property name="PI" value="3.1415926535897931"/>
   <xacro:property name="density" value="3.09"/>
-  <!-- <xacro:macro name="elfin3"> -->
-    <!-- TRANSMISSION: -->
-    <!-- <xacro:elfin3_transmission /> -->
-    <!-- GAZEBO - ROS2_CONTROL: -->
-    <!-- <xacro:elfin3_gazebo
-    use_real_hardware="$(arg use_real_hardware)"
-    use_fake_hardware="$(arg use_fake_hardware)"/> -->
   <link name="world"/>
   <joint name="world_base" type="fixed">
@@ -40,37 +30,37 @@
     <inertial>
       <origin
-        xyz="-0.000275485599623298 7.59034702891903E-06 0.0267651528589008"
-        rpy="0 0 0" />
-      <mass
-        value="0.728456071678781" />
-      <inertia
-        ixx="0.000970397629421624"
-        ixy="3.62553999566492E-08"
-        ixz="-1.47235460345842E-05"
-        iyy="0.00088280791320513"
-        iyz="-5.96416765248893E-08"
-        izz="0.00145846071899871" />
-    </inertial>
-    <visual>
-      <origin
-        xyz="0 0 0"
-        rpy="0 0 0" />
-      <geometry>
-        <mesh
-          filename="file://$(find elfin_description)/meshes/elfin3/elfin_base.STL" />
-      </geometry>
-      <material
-        name="">
-        <color
-          rgba="0.752941176470588 0.752941176470588 0.752941176470588 1" />
-      </material>
-    </visual>
-    <collision>
-      <origin
-        xyz="0 0 0"
-        rpy="0 0 0" />
-      <geometry>
-        <mesh
-          filename="file://$(find elfin_description)/meshes/elfin3/elfin_base.STL" />
+        xyz="0.00425937844813294 -0.000389571231902992 0.00274262778667868"
+        rpy="0 0 0" />
+      <mass
+        value="0.0268461773395224" />
+      <inertia
+        ixx="2.66341322206443E-05"
+        ixy="5.51640996553045E-08"
+        ixz="2.21112209410463E-12"
+        iyy="2.67121402645769E-05"
+        iyz="-3.17722287525956E-12"
+        izz="5.30011200382481E-05" />
+    </inertial>
+    <visual>
+      <origin
+        xyz="0 0 0"
+        rpy="0 0 0" />
+      <geometry>
+        <mesh
+          filename="file://$(find elfin_description)/meshes/elfin3/base_link.STL" />
+      </geometry>
+      <material
+        name="">
+        <color
+          rgba="0.686274509803922 0.686274509803922 0.686274509803922 1" />
+      </material>
+    </visual>
+    <collision>
+      <origin
+        xyz="0 0 0"
+        rpy="0 0 0" />
+      <geometry>
+        <mesh
+          filename="file://$(find elfin_description)/meshes/elfin3/base_link.STL" />
       </geometry>
     </collision>
@@ -80,15 +70,15 @@
     <inertial>
       <origin
-        xyz="-8.22323356984713E-06 -0.0039667333981909 -0.0290082756012436"
-        rpy="0 0 0" />
-      <mass
-        value="1.98577153801731" />
-      <inertia
-        ixx="0.0059460417373412"
-        ixy="-7.00618460961318E-07"
-        ixz="-2.70118506895605E-07"
-        iyy="0.00528005523214319"
-        iyz="0.00114506851258069"
-        izz="0.00325219340192972" />
+        xyz="-1.11474311817293E-05 -0.019295238440266 0.081643413279284"
+        rpy="0 0 0" />
+      <mass
+        value="1.52628719338585" />
+      <inertia
+        ixx="0.006028902112623"
+        ixy="-5.48816506919481E-07"
+        ixz="-2.73302311360408E-07"
+        iyy="0.00509895338088794"
+        iyz="0.00146640275062038"
+        izz="0.0028687934642813" />
     </inertial>
     <visual>
@@ -103,5 +93,5 @@
         name="">
         <color
-          rgba="0.752941176470588 0.752941176470588 0.752941176470588 1" />
+          rgba="0.772549019607843 0.752941176470588 0.733333333333333 1" />
       </material>
     </visual>
@@ -120,5 +110,5 @@
     type="revolute">
     <origin
-      xyz="0 0 0.1925"
+      xyz="0 0 0.0695"
       rpy="0 0 0" />
     <parent
@@ -126,178 +116,4 @@
     <child
       link="elfin_link1" />
-    <axis
-      xyz="0 0 1" />
-    <limit
-      lower="-3.14"
-      upper="3.14"
-      effort="200"
-      velocity="1.57" />
-  </joint>
-  <link
-    name="elfin_link2">
-    <inertial>
-      <origin
-        xyz="-1.16232734714673E-05 0.116434226200619 0.107577852399745"
-        rpy="0 0 0" />
-      <mass
-        value="1.40617433597616" />
-      <inertia
-        ixx="0.0116524684265068"
-        ixy="2.47639007244578E-06"
-        ixz="-1.30890011077188E-07"
-        iyy="0.000937691661869045"
-        iyz="0.000516659498705414"
-        izz="0.0120822102121993" />
-    </inertial>
-    <visual>
-      <origin
-        xyz="0 0 0"
-        rpy="0 0 0" />
-      <geometry>
-        <mesh
-          filename="file://$(find elfin_description)/meshes/elfin3/elfin_link2.STL" />
-      </geometry>
-      <material
-        name="">
-        <color
-          rgba="0.752941176470588 0.752941176470588 0.752941176470588 1" />
-      </material>
-    </visual>
-    <collision>
-      <origin
-        xyz="0 0 0"
-        rpy="0 0 0" />
-      <geometry>
-        <mesh
-          filename="file://$(find elfin_description)/meshes/elfin3/elfin_link2.STL" />
-      </geometry>
-    </collision>
-  </link>
-  <joint
-    name="elfin_joint2"
-    type="revolute">
-    <origin
-      xyz="0 0 0"
-      rpy="1.5708 0 0" />
-    <parent
-      link="elfin_link1" />
-    <child
-      link="elfin_link2" />
-    <axis
-      xyz="0 0 1" />
-    <limit
-      lower="-2.35"
-      upper="2.35"
-      effort="200"
-      velocity="1.57" />
-  </joint>
-  <link
-    name="elfin_link3">
-    <inertial>
-      <origin
-        xyz="0.0262387073150999 5.37044335293884E-06 -0.00343411596931149"
-        rpy="0 0 0" />
-      <mass
-        value="1.39255453742279" />
-      <inertia
-        ixx="0.00182232495944746"
-        ixy="-2.21097754348067E-07"
-        ixz="-0.000639319275242194"
-        iyy="0.00336261409093928"
-        iyz="-5.59685465899292E-07"
-        izz="0.0029273181824904" />
-    </inertial>
-    <visual>
-      <origin
-        xyz="0 0 0"
-        rpy="0 0 0" />
-      <geometry>
-        <mesh
-          filename="file://$(find elfin_description)/meshes/elfin3/elfin_link3.STL" />
-      </geometry>
-      <material
-        name="">
-        <color
-          rgba="0.752941176470588 0.752941176470588 0.752941176470588 1" />
-      </material>
-    </visual>
-    <collision>
-      <origin
-        xyz="0 0 0"
-        rpy="0 0 0" />
-      <geometry>
-        <mesh
-          filename="file://$(find elfin_description)/meshes/elfin3/elfin_link3.STL" />
-      </geometry>
-    </collision>
-  </link>
-  <joint
-    name="elfin_joint3"
-    type="revolute">
-    <origin
-      xyz="0 0.266 0"
-      rpy="3.1416 0 1.5708" />
-    <parent
-      link="elfin_link2" />
-    <child
-      link="elfin_link3" />
-    <axis
-      xyz="0 0 1" />
-    <limit
-      lower="-2.61"
-      upper="2.61"
-      effort="200"
-      velocity="1.57" />
-  </joint>
-  <link
-    name="elfin_link4">
-    <inertial>
-      <origin
-        xyz="1.95216712879575E-06 -0.0600119802928874 0.203829262782307"
-        rpy="0 0 0" />
-      <mass
-        value="1.01776198349465" />
-      <inertia
-        ixx="0.00655093186907593"
-        ixy="3.55081363904659E-08"
-        ixz="-4.08511113735521E-09"
-        iyy="0.00535736774588743"
-        iyz="0.00190350389406001"
-        izz="0.00209832030530978" />
-    </inertial>
-    <visual>
-      <origin
-        xyz="0 0 0"
-        rpy="0 0 0" />
-      <geometry>
-        <mesh
-          filename="file://$(find elfin_description)/meshes/elfin3/elfin_link4.STL" />
-      </geometry>
-      <material
-        name="">
-        <color
-          rgba="0.752941176470588 0.752941176470588 0.752941176470588 1" />
-      </material>
-    </visual>
-    <collision>
-      <origin
-        xyz="0 0 0"
-        rpy="0 0 0" />
-      <geometry>
-        <mesh
-          filename="file://$(find elfin_description)/meshes/elfin3/elfin_link4.STL" />
-      </geometry>
-    </collision>
-  </link>
-  <joint
-    name="elfin_joint4"
-    type="revolute">
-    <origin
-      xyz="0 0 0"
-      rpy="1.5708 0 1.5708" />
-    <parent
-      link="elfin_link3" />
-    <child
-      link="elfin_link4" />
     <axis
       xyz="0 0 1" />
@@ -309,18 +125,192 @@
   </joint>
   <link
+    name="elfin_link2">
+    <inertial>
+      <origin
+        xyz="-3.09813419838078E-05 -0.0392725728395098 0.121906520746464"
+        rpy="0 0 0" />
+      <mass
+        value="0.519379765009091" />
+      <inertia
+        ixx="0.00462941997584524"
+        ixy="9.53033193206284E-08"
+        ixz="1.89958745191593E-06"
+        iyy="0.00485416387879526"
+        iyz="-0.00019166604937554"
+        izz="0.000506978474454832" />
+    </inertial>
+    <visual>
+      <origin
+        xyz="0 0 0"
+        rpy="0 0 0" />
+      <geometry>
+        <mesh
+          filename="file://$(find elfin_description)/meshes/elfin3/elfin_link2.STL" />
+      </geometry>
+      <material
+        name="">
+        <color
+          rgba="0.501960784313725 0.501960784313725 0.501960784313725 1" />
+      </material>
+    </visual>
+    <collision>
+      <origin
+        xyz="0 0 0"
+        rpy="0 0 0" />
+      <geometry>
+        <mesh
+          filename="file://$(find elfin_description)/meshes/elfin3/elfin_link2.STL" />
+      </geometry>
+    </collision>
+  </link>
+  <joint
+    name="elfin_joint2"
+    type="revolute">
+    <origin
+      xyz="0 -0.066 0.123"
+      rpy="0 0 0" />
+    <parent
+      link="elfin_link1" />
+    <child
+      link="elfin_link2" />
+    <axis
+      xyz="0 -1 0" />
+    <limit
+      lower="-2.35"
+      upper="2.35"
+      effort="104"
+      velocity="1.27" />
+  </joint>
+  <link
+    name="elfin_link3">
+    <inertial>
+      <origin
+        xyz="7.94789705792241E-06 0.0434911461385148 0.0377663456053925"
+        rpy="0 0 0" />
+      <mass
+        value="1.07924103107593" />
+      <inertia
+        ixx="0.00347290093864989"
+        ixy="-5.5219540256932E-07"
+        ixz="-1.81596933237452E-07"
+        iyy="0.0028883932232078"
+        iyz="-0.000859331225721596"
+        izz="0.00165138765596417" />
+    </inertial>
+    <visual>
+      <origin
+        xyz="0 0 0"
+        rpy="0 0 0" />
+      <geometry>
+        <mesh
+          filename="file://$(find elfin_description)/meshes/elfin3/elfin_link3.STL" />
+      </geometry>
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
Commit message: exchange the position of tool_link and elfin_end_link

File: elfin3/elfin3_ros2_gazebo/urdf/elfin3.urdf.xacro (robot description, xacro)
@@ -424,8 +424,31 @@
       velocity="1.57" />
   </joint>
-  <link
-    name="elfin_end_link"/>
-  <joint
-    name="elfin_end_joint"
+  <link name="tool_link">
+    <inertial>
+      <origin xyz="0 0 0.7065" rpy="0 0 0"/>
+      <mass value="0.1"/>
+      <inertia
+        ixx="0.000016666" ixy="0.0" ixz="0.0"
+        iyy="0.000016666" iyz="0.0"
+        izz="0.000016666"/>
+    </inertial>
+    <visual>
+      <origin xyz="0 0 0.055" rpy="0 0 0"/>
+      <geometry>
+        <cylinder radius="0.01" length="0.11"/>
+      </geometry>
+      <material name="tool_color">
+        <color rgba="0.8 0.2 0.2 1.0"/>
+      </material>
+    </visual>
+    <collision>
+      <origin xyz="0 0 0.055" rpy="0 0 0"/>
+      <geometry>
+        <cylinder radius="0.01" length="0.11"/>
+      </geometry>
+    </collision>
+  </link>
+  <joint
+    name="tool_joint"
     type="fixed">
     <origin
@@ -435,31 +458,17 @@
       link="elfin_link6" />
     <child
-      link="elfin_end_link" />
+      link="tool_link" />
     <axis
       xyz="0 0 0" />
   </joint>
   <!-- Add tool link -->
-<link name="tool_link">
-  <visual>
-    <origin xyz="0 0 0" rpy="0 0 0"/>
-    <!-- <geometry>
-      <mesh filename="file://$(find your_package)/meshes/tool.stl"/>
-    </geometry> -->
-    <material name="tool_color">
-      <color rgba="0.8 0.2 0.2 1.0"/>
-    </material>
-  </visual>
-  <collision>
-    <origin xyz="0 0 0" rpy="0 0 0"/>
-    <!-- <geometry>
-      <mesh filename="file://$(find your_package)/meshes/tool.stl"/>
-    </geometry> -->
-  </collision>
+<link name="elfin_end_link">
+  <origin xyz="0 0 0.11" rpy="0 0 0"/>
 </link>
 <!-- Add tool joint -->
-<joint name="tool_joint" type="fixed">
-  <origin xyz="0 0 0.11" rpy="0 0 0"/>  <!-- 沿Z轴偏移110mm -->
-  <parent link="elfin_end_link"/>
-  <child link="tool_link"/>
+<joint name="elfin_end_joint" type="fixed">
+  <origin xyz="0 0 0.11" rpy="0 0 0"/>
+  <parent link="tool_link"/>
+  <child link="elfin_end_link"/>
 </joint>
 </robot>

Commit message: add a sensor_link with sensor joint

File: elfin3/elfin3_ros2_gazebo/urdf/elfin3.urdf.xacro (robot description, xacro)
@@ -472,3 +472,12 @@
   <child link="elfin_end_link"/>
 </joint>
+<!-- Add sensor link -->
+<link name="sensor_link">
+  <origin xyz="0 0 0" rpy="0 0 0"/>
+</link>
+<joint name="sensor_joint" type="fixed">
+  <origin xyz="0 0 0" rpy="0 0 -1.19163521"/>
+  <parent link="elfin_end_link"/>
+  <child link="sensor_link"/>
+</joint>
 </robot>
